File: blink/blink.kicad_pcb (KiCad board)
At the start: 2 copper layers, 27.6 x 24.3 mm, 2 parts

Commit message: Add 2nd LED
Parts:
- moved D1 6.12 mm to (156.8, 80.3)
- moved R1 6.12 mm to (162.5, 81.4)
Changed lines of the file:
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@@
   )
   (module Resistor_THT:R_Axial_DIN0204_L3.6mm_D1.6mm_P1.90mm_Vertical (layer F.Cu)
-    (at 157.7 85.2 90)
+    (at 162.5 81.4 90)
     (descr "Resistor, Axial_DIN0204 series, Axial, Vertical, pin pitch=1.9mm, 0.167W, length*diameter=3.6*1.6mm^2, http://cdn-reichelt.de/documents/datenblatt/B400/1_4W%23YAG.pdf")
     (tags "Resistor Axial_DIN0204 series Axial Vertical pin pitch 1.9mm 0.167W length 3.6mm diameter 1.6mm")
@@
       (effects (font (size 1 1) (thickness 0.15)))
     )
+    (fp_line (start 2.86 -1.05) (end -1.05 -1.05) (layer F.CrtYd) (width 0.05))
+    (fp_line (start 2.86 1.05) (end 2.86 -1.05) (layer F.CrtYd) (width 0.05))
+    (fp_line (start -1.05 1.05) (end 2.86 1.05) (layer F.CrtYd) (width 0.05))
+    (fp_line (start -1.05 -1.05) (end -1.05 1.05) (layer F.CrtYd) (width 0.05))
+    (fp_line (start 0 0) (end 1.9 0) (layer F.Fab) (width 0.1))
+    (fp_circle (center 0 0) (end 0.8 0) (layer F.Fab) (width 0.1))
     (fp_text user %R (at 0.95 -1.92 90) (layer F.Fab)
       (effects (font (size 1 1) (thickness 0.15)))
     )
     (fp_arc (start 0 0) (end 0.417133 -0.7) (angle -233.92106) (layer F.SilkS) (width 0.12))
-    (fp_circle (center 0 0) (end 0.8 0) (layer F.Fab) (width 0.1))
-    (fp_line (start 0 0) (end 1.9 0) (layer F.Fab) (width 0.1))
-    (fp_line (start -1.05 -1.05) (end -1.05 1.05) (layer F.CrtYd) (width 0.05))
-    (fp_line (start -1.05 1.05) (end 2.86 1.05) (layer F.CrtYd) (width 0.05))
-    (fp_line (start 2.86 1.05) (end 2.86 -1.05) (layer F.CrtYd) (width 0.05))
-    (fp_line (start 2.86 -1.05) (end -1.05 -1.05) (layer F.CrtYd) (width 0.05))
     (pad 2 thru_hole oval (at 1.9 0 90) (size 1.4 1.4) (drill 0.7) (layers *.Cu *.Mask)
       (net 3 GND))
@@
   )
   (module LED_SMD:LED_1206_3216Metric (layer F.Cu)
-    (at 152 84.1 90)
+    (at 156.8 80.3 90)
     (descr "LED SMD 1206 (3216 Metric), square (rectangular) end terminal, IPC_7351 nominal, (Body size source: http://www.tortai-tech.com/upload/download/2011102023233369053.pdf), generated with kicad-footprint-generator")
     (tags LED)
@@
       (effects (font (size 1 1) (thickness 0.15)))
     )
+    (fp_line (start 2.28 1.12) (end -2.28 1.12) (layer F.CrtYd) (width 0.05))
+    (fp_line (start 2.28 -1.12) (end 2.28 1.12) (layer F.CrtYd) (width 0.05))
+    (fp_line (start -2.28 -1.12) (end 2.28 -1.12) (layer F.CrtYd) (width 0.05))
+    (fp_line (start -2.28 1.12) (end -2.28 -1.12) (layer F.CrtYd) (width 0.05))
+    (fp_line (start -2.285 1.135) (end 1.6 1.135) (layer F.SilkS) (width 0.12))
+    (fp_line (start -2.285 -1.135) (end -2.285 1.135) (layer F.SilkS) (width 0.12))
+    (fp_line (start 1.6 -1.135) (end -2.285 -1.135) (layer F.SilkS) (width 0.12))
+    (fp_line (start 1.6 0.8) (end 1.6 -0.8) (layer F.Fab) (width 0.1))
+    (fp_line (start -1.6 0.8) (end 1.6 0.8) (layer F.Fab) (width 0.1))
+    (fp_line (start -1.6 -0.4) (end -1.6 0.8) (layer F.Fab) (width 0.1))
+    (fp_line (start -1.2 -0.8) (end -1.6 -0.4) (layer F.Fab) (width 0.1))
+    (fp_line (start 1.6 -0.8) (end -1.2 -0.8) (layer F.Fab) (width 0.1))
     (fp_text user %R (at 0 0 90) (layer F.Fab)
       (effects (font (size 0.8 0.8) (thickness 0.12)))
     )
-    (fp_line (start 1.6 -0.8) (end -1.2 -0.8) (layer F.Fab) (width 0.1))
-    (fp_line (start -1.2 -0.8) (end -1.6 -0.4) (layer F.Fab) (width 0.1))
-    (fp_line (start -1.6 -0.4) (end -1.6 0.8) (layer F.Fab) (width 0.1))
-    (fp_line (start -1.6 0.8) (end 1.6 0.8) (layer F.Fab) (width 0.1))
-    (fp_line (start 1.6 0.8) (end 1.6 -0.8) (layer F.Fab) (width 0.1))
-    (fp_line (start 1.6 -1.135) (end -2.285 -1.135) (layer F.SilkS) (width 0.12))
-    (fp_line (start -2.285 -1.135) (end -2.285 1.135) (layer F.SilkS) (width 0.12))
-    (fp_line (start -2.285 1.135) (end 1.6 1.135) (layer F.SilkS) (width 0.12))
-    (fp_line (start -2.28 1.12) (end -2.28 -1.12) (layer F.CrtYd) (width 0.05))
-    (fp_line (start -2.28 -1.12) (end 2.28 -1.12) (layer F.CrtYd) (width 0.05))
-    (fp_line (start 2.28 -1.12) (end 2.28 1.12) (layer F.CrtYd) (width 0.05))
-    (fp_line (start 2.28 1.12) (end -2.28 1.12) (layer F.CrtYd) (width 0.05))
     (pad 2 smd roundrect (at 1.4 0 90) (size 1.25 1.75) (layers F.Cu F.Paste F.Mask) (roundrect_rratio 0.2)
       (net 1 +5V))
@@
   (gr_line (start 171.8 70.6) (end 171.8 94.9) (layer Edge.Cuts) (width 0.05))
   (gr_line (start 144.2 70.6) (end 171.8 70.6) (layer Edge.Cuts) (width 0.05))
-  (segment (start 157.4 85.5) (end 157.7 85.2) (width 0.25) (layer F.Cu) (net 2))
-  (segment (start 152 85.5) (end 157.4 85.5) (width 0.25) (layer F.Cu) (net 2))
+  (segment (start 162.2 81.7) (end 162.5 81.4) (width 0.25) (layer F.Cu) (net 2))
+  (segment (start 156.8 81.7) (end 162.2 81.7) (width 0.25) (layer F.Cu) (net 2))
 )
